File: HARDWARE/GATE2TRIG.kicad_pcb (KiCad board)
At the start: 2 copper layers, 45 x 175 mm, 43 parts, among them J1 Gate3in, J10 Gate-1, J11 Gate-2, J12 Gate-3, J13 Gate-4, J2 Gate1in, J3 Gate4in, J4 TRIG-2, J5 Gate2in, J6 Conn_02x05_Odd_Even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

Commit message: PICS
Other:
- board text added: "FIT ONLY R1 or RV1 ( R1 TBD)"
- board text added: "GATE-2-TRIGER V1.0.0 By TwinTurbo"
- board text added: "V1.0.0"
