File: HARDWARE/GATE2TRIG.sch (KiCad schematic (older format))
At the start: 42 parts, among them J1 Gate3in, J10 Gate-1, J11 Gate-2, J12 Gate-3, J13 Gate-4, J2 Gate1in, J3 Gate4in, J4 TRIG-2, J5 Gate2in, J6 Conn_02x05_Odd_Even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

Commit message: PICS
Other:
- note added: "13/07/2020 -- TwinTurbo V1.0.0"
- note removed: "DRAF UNTRESTED 13/07/2020 -- TwinTurbo"
Changed lines of the file:
@@
 Connection ~ 7150 4500
 Text Notes 7100 7100 0    118  ~ 0
-DRAF UNTRESTED 13/07/2020 -- TwinTurbo
+13/07/2020 -- TwinTurbo V1.0.0
 $EndSCHEMATC

Commit message: holidaysync
Other:
- note added: "22/02/2022 -- TwinTurbo V1.0.0"
- note removed: "13/07/2020 -- TwinTurbo V1.0.0"
Changed lines of the file:
@@
 Connection ~ 7150 4500
 Text Notes 7100 7100 0    118  ~ 0
-13/07/2020 -- TwinTurbo V1.0.0
+22/02/2022 -- TwinTurbo V1.0.0
 $EndSCHEMATC
