File: HARDWARE/Front/Panel.kicad_pcb (KiCad board)
At the start: 2 copper layers, 383.5 x 264 mm, 23 parts, among them SW9 RUNSTOP

Commit message: PICS
Parts:
- removed +12V: LED +12, RobsFoots:FP-LED_D5.0mm
- removed -12V: LED -12, RobsFoots:FP-LED_D5.0mm
- removed the G*** at (6.60, 80.5)
- removed the H1 at (459.2, -40.5)
- removed the H1 at (180.9, 152.0)
- removed the H1 at (137.9, 152.0)
- removed the H1 at (137.9, -41.0)
- removed the H1 at (100.7, 215.2)
- removed the H1 at (82.7, 215.2)
- removed the H1 at (82.7, 22.2)
- removed the H1 at (40.9, 172.0)
- removed the H1 at (54.4, 109.0)
- removed the H1 at (100.7, 22.2)
- removed the H1 at (366.2, 152.5)
- removed the H1 at (366.2, -40.5)
- removed the H1 at (459.2, 152.5)
- removed the H1 at (297.0, 151.2)
- removed the H1 at (297.0, -41.8)
- removed the H1 at (229.0, 151.2)
- removed the H1 at (229.0, -41.8)
- removed the H1 at (180.9, -41.0)
- removed SW9: RUNSTOP, RobsFoots:FP-MINITOGLE
- added G***: LOGO, ROBSLIBRARY:TOBINLOGO, B.Cu at (181.6, 134.0)
- added G***: LOGO, ROBSLIBRARY:K6neg, B.Cu at (170.9, 61.2)
- added H1: MountingHole_Pad, MountingHole:MountingHole_3.2mm_M3_DIN965_Pad, F.Cu at (148.5, -17.5)
- added H1: MountingHole_Pad, MountingHole:MountingHole_3.2mm_M3_DIN965_Pad, F.Cu at (191.5, 175.5)
- added H1: MountingHole_Pad, MountingHole:MountingHole_3.2mm_M3_DIN965_Pad, F.Cu at (191.5, -17.5)
- added H1: MountingHole_Pad, MountingHole:MountingHole_3.2mm_M3_DIN965_Pad, F.Cu at (148.5, 175.5)
- added J1: Gate3in, ROBSLIBRARY:PANEL-LMNC, F.Cu at (158.1, 84.2)
- added J10: Gate-1, ROBSLIBRARY:PANEL-LMNC, F.Cu at (158.1, 18.2)
- added J11: Gate-2, ROBSLIBRARY:PANEL-LMNC, F.Cu at (158.1, 62.2)
- added J12: Gate-3, ROBSLIBRARY:PANEL-LMNC, F.Cu at (158.1, 106.2)
- added J13: Gate-4, ROBSLIBRARY:PANEL-LMNC, F.Cu at (158.1, 150.2)
- added J2: Gate1in, ROBSLIBRARY:PANEL-LMNC, F.Cu at (158.1, -3.83)
- added J3: Gate4in, ROBSLIBRARY:PANEL-LMNC, F.Cu at (158.1, 128.2)
- added J4: TRIG-2, ROBSLIBRARY:PANEL-LMNC, F.Cu at (183.1, 62.2)
- added J5: Gate2in, ROBSLIBRARY:PANEL-LMNC, F.Cu at (158.1, 40.2)
- added J7: TRIG-1, ROBSLIBRARY:PANEL-LMNC, F.Cu at (183.1, 18.2)
- added J8: TRIG-3, ROBSLIBRARY:PANEL-LMNC, F.Cu at (183.1, 106.2)
- added J9: TRIG-4, ROBSLIBRARY:PANEL-LMNC, F.Cu at (183.1, 150.2)
- added REF**: 20K 3296W, AA-ROB-FULL:PannelBournTrimmer-no3d, F.Cu at (176.4, 7.67)
- moved G*** 222.4 mm to (183.9, 0.81), turned to 180 degrees
Routing:
- net (no net): track 0.00 -> 1.06 mm
Other:
- board size 383.5 x 264 mm -> 50 x 200 mm
- board text added: "1"
- board text added: "2"
- board text added: "3"
- board text added: "4"
- board text added: "By Twin Turbo"
- board text added: "C H N 3"
- board text added: "CLAYTUNE - Simple GATE TO TRIGGER V1.0 - By TwinTurbo"
- board text added: "For Kate"
- board text added: "GATE IN"
- board text added: "GATE OUT"
- board text added: "JLCJLCJLCJLC"
- board text added: "Quad Gate To Trigger"
- board text added: "TRIGGER"
- board text added: "The Lloyd-Pack"
- board text removed: "BIG RED BUSS"
- board text removed: "Big Red Buss- PCB V 0.1.0"
- board text removed: "CLAYTUNE - Big Red Buss V0.1.0 - By TwinTurbo - JLCJLCJLCJLC"
- board text removed: "CLAYTUNE Big Red Buss By TwinTurbo"
- board text removed: "For Kate By TwinTurbo"
- board text removed: "OFF"
- board text removed: "ON"
